File: SeniorDesign_Block2_ADC/_autosave-SeniorDesign_Block2_ADC.sch (KiCad schematic (older format))
At the start: 32 parts, among them J1 Conn_02x18_Row_Letter_First, J10 Conn_01x01, J11 Conn_01x08, J12 Conn_01x01, J2 Conn_02x18_Row_Letter_First, J3 Conn_01x02_Male, J4 Conn_01x02_Male, J5 Conn_01x01, J6 Conn_01x01, J7 Conn_01x01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

Commit message: Continued work.  Push to github.  Even worse commit messages.
Parts:
- gave numbers to parts that had none: 1
Changed lines of the file:
@@
 conn_gnd
 $Comp
-L Connector_Generic:Conn_01x01 J?
+L Connector_Generic:Conn_01x01 J13
 U 1 1 602CBBD8
 P 1550 4950
-F 0 "J?" H 1468 4725 50  0000 C CNN
+F 0 "J13" H 1468 4725 50  0000 C CNN
 F 1 "Conn_01x01" H 1468 4816 50  0000 C CNN
 F 2 "Connector_PinHeader_2.54mm:PinHeader_1x01_P2.54mm_Vertical" H 1550 4950 50  0001 C CNN
